Commit message: Update the URDF with geometries provided by Stuart, also collision and inertia are updated accordingly.

File: urdf/alkimia_door.urdf.xacro (robot description, xacro)
@@ -10,21 +10,21 @@
 			<parent link="${parent}"/>
 			<child link="${name}_top_fin"/>
-			<axis xyz="0 0 1" />
+			<axis xyz="1 0 0" />
 			<limit lower="${0*pi/180}" upper="${85*pi/180}" effort="60" velocity="10"/>
 		</joint>
 		<link name="${name}_top_fin">
 			<inertial>
-				<origin xyz="0.5 0.005 0.15" rpy="0 0 0"/>
+				<origin xyz="-0.1 -0.55 0.01" rpy="0 0 0"/>
 				<mass value="2.0"/>
 				<inertia
-				ixx="0.06" ixy="0.0" ixz="0.0"
-				iyy="2.7" iyz="0.0"
+				ixx="2.6" ixy="0.0" ixz="0.0"
+				iyy="0.06" iyz="0.0"
 				izz="2.6"/>
 			</inertial>
 			<visual>
-				<origin xyz="0.5 0 0.15" rpy="0 0 0" />
+				<origin xyz="0 0 0" rpy="0 0 0" />
 				<geometry>
-					<!-- mesh filename="package://alkimia_door/urdf/meshes/top_fin.stl" scale=" .001 .001 .001" / -->
-					<box size="1.0 0.01 0.3"/>
+					<mesh filename="package://alkimia_door/urdf/meshes/top_fin.stl" scale=" .001 .001 .001" />
+					<!-- box size="1.0 0.01 0.3"/ -->
 				</geometry>
 				<material name="Brown">
@@ -33,8 +33,8 @@
 			</visual>
 			<collision>
-				<origin xyz="0.5 0 0.15" rpy="0 0 0" />
+				<origin xyz="-0.1 -0.55 0.01" rpy="0 0 0" />
 				<geometry>
 					<!-- mesh filename="package://alkimia_door/urdf/meshes/top_fin.stl" scale=" .001 .001 .001" / -->
-					<box size="1.0 0.01 0.3"/>
+					<box size="0.2 1.1 0.02"/>
 				</geometry>
 			</collision>
@@ -42,5 +42,5 @@
 		<!-- BOTTOM FIN -->
 		<joint name="${name}_bottom_joint" type="revolute">
-			<origin xyz="1.0 0.0 0.0" rpy="0.0 0.0 0.0" />
+			<origin xyz="0.0 -1.11 0.0" rpy="-1.57 0 -1.57" />
 			<parent link="${name}_top_fin"/>
 			<child link="${name}_bottom_fin"/>
@@ -53,16 +53,16 @@
 		<link name="${name}_bottom_fin">
 			<inertial>
-				<origin xyz="0.5 0.005 0.15" rpy="0 0 0"/>
+				<origin xyz="0.35 -0.01 -0.1" rpy="0 0 0"/>
 				<mass value="1.0"/>
 				<inertia
 				ixx="0.03" ixy="0.0" ixz="0.0"
-				iyy="1.35" iyz="0.0"
+				iyy="1.3" iyz="0.0"
 				izz="1.3"/>
 			</inertial>
 			<visual>
-				<origin xyz="0.5 0 0.15" rpy="0 0 0" />
+				<origin xyz="0.07 0.12 -0.017" rpy="0 0 0" />
 				<geometry>
-					<!-- mesh filename="package://alkimia_door/urdf/meshes/bottom_fin.stl" scale=" .001 .001 .001" / -->
-					<box size="1.0 0.01 0.3"/>
+					<mesh filename="package://alkimia_door/urdf/meshes/bottom_fin.stl" scale=" .001 .001 .001" />
+					<!-- box size="1.0 0.01 0.3"/ -->
 				</geometry>
 				<material name="Brown">
@@ -71,8 +71,8 @@
 			</visual>
 			<collision>
-				<origin xyz="0.5 0 0.15" rpy="0 0 0" />
+				<origin xyz="0.65 -0.01 -0.1" rpy="0 0 0" />
 				<geometry>
 					<!-- mesh filename="package://alkimia_door/urdf/meshes/bottom_fin.stl" scale=" .001 .001 .001" / -->
-					<box size="1.0 0.01 0.3"/>
+					<box size="1.3 0.02 0.2"/>
 				</geometry>
 			</collision>
@@ -98,11 +98,12 @@
 	</xacro:macro>
 	<link name="world"/>
-	<joint name="anchor_joint" type="fixed">
+	<joint name="anchor_joint1" type="fixed">
+		<origin xyz="0 0 0" rpy="0 0 0"/>
 		<parent link="world"/>
-		<child link="Iprofile"/>
+		<child link="Iprofile1"/>
 	</joint>
-	<link name="Iprofile">
+	<link name="Iprofile1">
 		<inertial>
-			<origin xyz="0.5 0.005 0.15" rpy="0 0 0"/>
+			<origin xyz="0 0 -0.1" rpy="0 0 0"/>
 			<mass value="50.0"/>
 			<inertia
@@ -112,7 +113,8 @@
 		</inertial>
 		<visual>
-			<origin xyz="-0.1 -0.1 2.55" rpy="0.0 0 0"/>
+			<origin xyz="0 0 0" rpy="0.0 0 0"/>
 			<geometry>
-				<box size="0.2 0.2 5.1"/>
+				<mesh filename="package://alkimia_door/urdf/meshes/roof.stl" scale=" .001 .001 .001" />
+				<!-- box size="0.2 0.2 5.1"/ -->
 			</geometry>
 			<material name="Gray">
@@ -121,12 +123,43 @@
 		</visual>
 		<collision>
-			<origin xyz="-0.1 -0.1 2.55" rpy="0.0 0 0"/>
+			<origin xyz="-0.1 -4 -0.1" rpy="0.0 0 0"/>
 			<geometry>
-				<box size="0.2 0.2 5.1"/>
+				<box size="0.2 8 0.2"/>
 			</geometry>
 		</collision>
 	</link>
-	<xacro:fin parent="Iprofile" name="fin1" position="0 0 0" orientation="0 0 0" isCoupled="${coupleFins}" ratio="2"/>
-	<xacro:fin parent="Iprofile" name="fin2" position="0 0 0.4" orientation="0 0 0" isCoupled="${coupleFins}" ratio="2"/>
+	<joint name="anchor_joint2" type="fixed">
+		<origin xyz="0 0 0.3" rpy="0 0 0"/>
+		<parent link="world"/>
+		<child link="Iprofile2"/>
+	</joint>
+	<link name="Iprofile2">
+		<inertial>
+			<origin xyz="0 0 -0.1" rpy="0 0 0"/>
+			<mass value="50.0"/>
+			<inertia
+			ixx="1.0" ixy="0.0" ixz="0.0"
+			iyy="1.0" iyz="0.0"
+			izz="1.0"/>
+		</inertial>
+		<visual>
+			<origin xyz="0 0 0" rpy="0.0 0 0"/>
+			<geometry>
+				<mesh filename="package://alkimia_door/urdf/meshes/roof.stl" scale=" .001 .001 .001" />
+				<!-- box size="0.2 0.2 5.1"/ -->
+			</geometry>
+			<material name="Gray">
+				<color rgba="0.5 0.5 0.5 1.0"/>
+			</material>
+		</visual>
+		<collision>
+			<origin xyz="-0.1 -4 -0.1" rpy="0.0 0 0"/>
+			<geometry>
+				<box size="0.2 8 0.2"/>
+			</geometry>
+		</collision>
+	</link>
+	<xacro:fin parent="Iprofile1" name="fin1" position="0.11 -0.13 -0.2" orientation="0 1.57 1.57" isCoupled="${coupleFins}" ratio="2"/>
+	<xacro:fin parent="Iprofile2" name="fin2" position="0.11 -0.13 -0.2" orientation="0 1.57 1.57" isCoupled="${coupleFins}" ratio="2"/>
 	<!-- <xacro:fin parent="Iprofile" name="fin3" position="0 0 0.6" orientation="0 0 0" isCoupled="${coupleFins}" ratio="2"/>
 	<xacro:fin parent="Iprofile" name="fin4" position="0 0 0.9" orientation="0 0 0" isCoupled="${coupleFins}" ratio="2"/>

Commit message: Updates to deal with passively actuated joints coupled with torsional springs

File: urdf/alkimia_door.urdf.xacro (robot description, xacro)
@@ -2,7 +2,44 @@
 <robot xmlns:xacro="http://www.ros.org/wiki/xacro" name="alkimia_door">
 	<xacro:property name="pi" value="3.1415926535897931" />
-	<xacro:property name="coupleFins" value="false" />
+	<xacro:property name="coupleFins" value="true" />
+	<!-- Profile model -->
+	<xacro:macro name="profile" params="parent name position orientation">
+		<joint name="${name}_joint" type="fixed">
+			<origin xyz="${position}" rpy="${orientation}" />
+			<parent link="${parent}"/>
+			<child link="${name}"/>
+			<axis xyz="1 0 0" />
+			<limit lower="${0*pi/180}" upper="${90*pi/180}" effort="60" velocity="10"/>
+			<dynamics damping="1.0" friction="10.0"/>
+		</joint>
+		<link name="${name}">
+			<inertial>
+				<origin xyz="0 0 -0.1" rpy="0 0 0"/>
+				<mass value="50.0"/>
+				<inertia
+				ixx="1.0" ixy="0.0" ixz="0.0"
+				iyy="1.0" iyz="0.0"
+				izz="1.0"/>
+			</inertial>
+			<visual>
+				<origin xyz="0 0 0" rpy="0.0 0 0"/>
+				<geometry>
+					<mesh filename="package://alkimia_door/urdf/meshes/roof.stl" scale=" .001 .001 .001" />
+					<!-- box size="0.2 0.2 5.1"/ -->
+				</geometry>
+				<material name="Gray">
+					<color rgba="0.5 0.5 0.5 1.0"/>
+				</material>
+			</visual>
+			<collision>
+				<origin xyz="-0.1 -4 -0.1" rpy="0.0 0 0"/>
+				<geometry>
+					<box size="0.2 8 0.2"/>
+				</geometry>
+			</collision>
+		</link>
+	</xacro:macro>
 	<!-- FIN model -->
-	<xacro:macro name="fin" params="parent name position orientation isCoupled ratio">
+	<xacro:macro name="fin" params="parent name position orientation">
 		<!-- TOP FIN -->
 		<joint name="${name}_top_joint" type="revolute">
@@ -11,5 +48,6 @@
 			<child link="${name}_top_fin"/>
 			<axis xyz="1 0 0" />
-			<limit lower="${0*pi/180}" upper="${85*pi/180}" effort="60" velocity="10"/>
+			<limit lower="${0*pi/180}" upper="${90*pi/180}" effort="60" velocity="10"/>
+			<dynamics damping="1.0" friction="10.0"/>
 		</joint>
 		<link name="${name}_top_fin">
@@ -46,13 +84,11 @@
 			<child link="${name}_bottom_fin"/>
 			<axis xyz="0 0 -1" />
-			<limit lower="${0*pi/180}" upper="${160*pi/180}" effort="60" velocity="10"/>
-			<xacro:if value="${isCoupled}">
-				<mimic joint="${name}_top_joint" multiplier="${ratio}"/>
-			</xacro:if>
+			<limit lower="${0*pi/180}" upper="${180*pi/180}" effort="60" velocity="10"/>
+			<dynamics damping="0.5" friction="5.0"/>
 		</joint>
 		<link name="${name}_bottom_fin">
 			<inertial>
 				<origin xyz="0.35 -0.01 -0.1" rpy="0 0 0"/>
-				<mass value="1.0"/>
+				<mass value="1.5"/>
 				<inertia
 				ixx="0.03" ixy="0.0" ixz="0.0"
@@ -90,76 +126,26 @@
 			<type>transmission_interface/SimpleTransmission</type>
 			<joint name="${name}_bottom_joint">
-				<hardwareInterface>EffortJointInterface</hardwareInterface>
+				<hardwareInterface>PositionJointInterface</hardwareInterface>
 			</joint>
-			<actuator name="${name}_bottom_fin_motor">
-				<mechanicalReduction>1</mechanicalReduction>
+			<actuator name="${name}_top_fin_motor">
+				<mechanicalReduction>-2</mechanicalReduction>
 			</actuator>
 		</transmission>
 	</xacro:macro>
 	<link name="world"/>
-	<joint name="anchor_joint1" type="fixed">
-		<origin xyz="0 0 0" rpy="0 0 0"/>
-		<parent link="world"/>
-		<child link="Iprofile1"/>
-	</joint>
-	<link name="Iprofile1">
-		<inertial>
-			<origin xyz="0 0 -0.1" rpy="0 0 0"/>
-			<mass value="50.0"/>
-			<inertia
-			ixx="1.0" ixy="0.0" ixz="0.0"
-			iyy="1.0" iyz="0.0"
-			izz="1.0"/>
-		</inertial>
-		<visual>
-			<origin xyz="0 0 0" rpy="0.0 0 0"/>
-			<geometry>
-				<mesh filename="package://alkimia_door/urdf/meshes/roof.stl" scale=" .001 .001 .001" />
-				<!-- box size="0.2 0.2 5.1"/ -->
-			</geometry>
-			<material name="Gray">
-				<color rgba="0.5 0.5 0.5 1.0"/>
-			</material>
-		</visual>
-		<collision>
-			<origin xyz="-0.1 -4 -0.1" rpy="0.0 0 0"/>
-			<geometry>
-				<box size="0.2 8 0.2"/>
-			</geometry>
-		</collision>
-	</link>
-	<joint name="anchor_joint2" type="fixed">
-		<origin xyz="0 0 0.3" rpy="0 0 0"/>
-		<parent link="world"/>
-		<child link="Iprofile2"/>
-	</joint>
-	<link name="Iprofile2">
-		<inertial>
-			<origin xyz="0 0 -0.1" rpy="0 0 0"/>
-			<mass value="50.0"/>
-			<inertia
-			ixx="1.0" ixy="0.0" ixz="0.0"
-			iyy="1.0" iyz="0.0"
-			izz="1.0"/>
-		</inertial>
-		<visual>
-			<origin xyz="0 0 0" rpy="0.0 0 0"/>
-			<geometry>
-				<mesh filename="package://alkimia_door/urdf/meshes/roof.stl" scale=" .001 .001 .001" />
-				<!-- box size="0.2 0.2 5.1"/ -->
-			</geometry>
-			<material name="Gray">
-				<color rgba="0.5 0.5 0.5 1.0"/>
-			</material>
-		</visual>
-		<collision>
-			<origin xyz="-0.1 -4 -0.1" rpy="0.0 0 0"/>
-			<geometry>
-				<box size="0.2 8 0.2"/>
-			</geometry>
-		</collision>
-	</link>
-	<xacro:fin parent="Iprofile1" name="fin1" position="0.11 -0.13 -0.2" orientation="0 1.57 1.57" isCoupled="${coupleFins}" ratio="2"/>
-	<xacro:fin parent="Iprofile2" name="fin2" position="0.11 -0.13 -0.2" orientation="0 1.57 1.57" isCoupled="${coupleFins}" ratio="2"/>
+    <xacro:profile parent="world" name="Iprofile1" position="0.0 0.0 0.0" orientation="0.0 0.0 0.0" />
+	<xacro:fin parent="Iprofile1" name="fin1" position="0.11 -0.13 -0.2" orientation="0 1.57 1.57" />
+    <xacro:profile parent="world" name="Iprofile2" position="0.0 0.0 0.3" orientation="0.0 0.0 0.0" />
+	<xacro:fin parent="Iprofile2" name="fin2" position="0.11 -0.13 -0.2" orientation="0 1.57 1.57" />
+    <xacro:profile parent="world" name="Iprofile3" position="0.0 0.0 0.6" orientation="0.0 0.0 0.0" />
+	<xacro:fin parent="Iprofile3" name="fin3" position="0.11 -0.13 -0.2" orientation="0 1.57 1.57" />
+    <xacro:profile parent="world" name="Iprofile4" position="0.0 0.0 0.9" orientation="0.0 0.0 0.0" />
+	<xacro:fin parent="Iprofile4" name="fin4" position="0.11 -0.13 -0.2" orientation="0 1.57 1.57" />
+    <xacro:profile parent="world" name="Iprofile5" position="0.0 0.0 1.2" orientation="0.0 0.0 0.0" />
+	<xacro:fin parent="Iprofile5" name="fin5" position="0.11 -0.13 -0.2" orientation="0 1.57 1.57" />
+    <xacro:profile parent="world" name="Iprofile6" position="0.0 0.0 1.5" orientation="0.0 0.0 0.0" />
+	<xacro:fin parent="Iprofile6" name="fin6" position="0.11 -0.13 -0.2" orientation="0 1.57 1.57" />
+    <xacro:profile parent="world" name="Iprofile7" position="0.0 0.0 1.8" orientation="0.0 0.0 0.0" />
+	<xacro:fin parent="Iprofile7" name="fin7" position="0.11 -0.13 -0.2" orientation="0 1.57 1.57" />
 	<!-- <xacro:fin parent="Iprofile" name="fin3" position="0 0 0.6" orientation="0 0 0" isCoupled="${coupleFins}" ratio="2"/>
 	<xacro:fin parent="Iprofile" name="fin4" position="0 0 0.9" orientation="0 0 0" isCoupled="${coupleFins}" ratio="2"/>
@@ -178,5 +164,9 @@
 	<xacro:fin parent="Iprofile" name="fin17" position="0 0 4.8" orientation="0 0 0" isCoupled="${coupleFins}" ratio="2"/> -->
 	<gazebo>
-		<plugin name="gazebo_ros_control" filename="libgazebo_ros_control.so"/>
+		<plugin name="alkimia_plugins" filename="libalkimia_plugins.so">
+			<robotNamespace>alkimia_door</robotNamespace>
+			<master1>fin1</master1>
+			<couplingStiffness>150</couplingStiffness>
+		</plugin>
 	</gazebo>
 </robot>
